File: Fichiers Eagle/main.sch (EAGLE design)
At the start: 31 parts, among them U1 TL082P, U2 TL084P

Commit message: mise à jour cartouche Schematic
Other:
- note added: "Mathieu Cariou UBO Open Factory 12/01/2021"
Changed lines of the file:
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@@
 <plain>
 <wire x1="88.9" y1="63.5" x2="93.98" y2="63.5" width="0.1524" layer="94"/>
+<text x="139.7" y="-25.4" size="1.778" layer="91">Mathieu Cariou
+UBO Open Factory
+12/01/2021</text>
 </plain>
 <instances>
@@
 </drawing>
 <compatibility>
+<note version="6.3" minversion="6.2.2" severity="warning">
+Since Version 6.2.2 text objects can contain more than one line,
+which will not be processed correctly with this version.
+</note>
 <note version="8.2" severity="warning">
 Since Version 8.2, EAGLE supports online libraries. The ids
